File: apa102-controller.sch (EAGLE design)
At the start: 165 parts, among them IC1 REG1117, IC3 IC_MCP7940M-SOIC8, J1 DCJ0202, U1 ATMEGA328P, U2 74HC04_HEX_INVERTERSOIC, U3 24AA32A-I/MS, U4 ATMEGA328P, U5 TEXAS-INSTRUMENTS_BY_ELEMENT1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

Commit message: more labels
Parts:
- added LED12: CBUS0, adafruit:LEDCHIP-LED0805
- added R28: 1k, rcl:R-US_R0805
- C1: value 10 -> 1u
- C2: value 100 -> 100n
- LED1: value (none) -> PWR-5MM
- LED9: value (none) -> PPS
Connections:
- net ADC1 renamed ADC1_TRIMPOT
- net ADC2 renamed ADC2_TRIMPOT
- net ARD_D4 renamed ARD_D4_GPS_EN
- net ARD_D9 renamed D9_LED_RED
- net D5 renamed D5_LED_GREEN
- net D6 renamed D6_LED_WHITE
- net DMINUS renamed UBLOX_DMINUS
- net DPLUS renamed UBLOX_DPLUS
- net N$12 renamed GPS_SDA
- net N$49 renamed WIREPAD_D8
- net N$55 renamed FT_DM
- net N$56 renamed FT_DP
- net N$6 renamed WIREPAD_D7
- net N$7 renamed UBLOX_RF_IN
- net N$8 renamed VCC_RF_2
- net RESET_PIN renamed ISP_RESET
- net SCL renamed ARD_SCK
- net SDI_ONE renamed ARD_MOSI
- removed net N$10: C44.1, C49.1, R11.2, U$21.3V3OUT, U$21.RESET#, U$21.VCCIO
- new net FT230_VCCIO: C44.1, C49.1, R11.2, R28.2, U$21.3V3OUT, U$21.RESET#, U$21.VCCIO
- new net FT_CB0: LED12.C, U$21.CBUS0
- new net N$58: LED12.A, R28.1
- net GND: now also U$21.GND1, U$21.GND2, U$21.GND3
Other:
- note added: ""Connecting a 22nF between the BP pin and GND pin significantly reduces noise on the regulator output...""
- note added: "COM0: "Connect to GND to use USB in Self Powered mode""
- note removed: "COM0 "Connect to GND to use USB in Self Powered mode""
- note removed: "Connecting a 22nF between the BP pin and GND pin significantly reduces noise on the regulator output, it is critical that the capacitor connection between the BP pin and GND pin be direct and PCB traces should be as short as possible."
- moved on the sheet: C48, C49, D4, D5, D6, LED10, LED11, R10, R25, R30, R31, R9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

Commit message: pcbs 20170206
Parts:
- removed SJ1: (no value), jumper:SJ
Connections:
- removed net N$25: SJ1.2, U1.AREF
- net +5V: no longer SJ1.1
Changed lines of the file:
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@@
 <part name="C25" library="rcl" deviceset="C-US" device="C0805" value="100nF"/>
 <part name="GND3" library="supply1" deviceset="GND" device=""/>
-<part name="SJ1" library="jumper" deviceset="SJ" device=""/>
 <part name="U2" library="SparkFun-DigitalIC" deviceset="74HC04_HEX_INVERTER" device="SOIC"/>
 <part name="JP1" library="SparkFun-Connectors" deviceset="M03X2" device="SHROUD"/>
@@
 <instance part="C25" gate="G$1" x="685.8" y="48.26"/>
 <instance part="GND3" gate="1" x="685.8" y="40.64"/>
-<instance part="SJ1" gate="1" x="63.5" y="172.72"/>
 <instance part="U2" gate="G$1" x="238.76" y="50.8"/>
 <instance part="JP1" gate="G$1" x="53.34" y="12.7"/>
@@
 <wire x1="71.12" y1="182.88" x2="58.42" y2="182.88" width="0.1524" layer="91"/>
 <junction x="58.42" y="182.88"/>
-<wire x1="58.42" y1="172.72" x2="58.42" y2="177.8" width="0.1524" layer="91"/>
-<junction x="58.42" y="177.8"/>
-<pinref part="SJ1" gate="1" pin="1"/>
 <wire x1="58.42" y1="185.42" x2="60.96" y2="185.42" width="0.1524" layer="91"/>
 <wire x1="60.96" y1="185.42" x2="60.96" y2="190.5" width="0.1524" layer="91"/>
@@
 </segment>
 </net>
-<net name="N$25" class="0">
-<segment>
-<pinref part="U1" gate="G$1" pin="AREF"/>
-<wire x1="71.12" y1="172.72" x2="68.58" y2="172.72" width="0.1524" layer="91"/>
-<pinref part="SJ1" gate="1" pin="2"/>
-</segment>
-</net>

Commit message: add 1N4733 Zener
Parts:
- added D7: (no value), diode:ZENER-DIODEDO41Z10
- LED12: value CBUS0 -> CBUS1
Connections:
- net N$26 renamed USB_RAW_5V
- net +5V: now also D7.C
- net FT_CB0: now also U$21.CBUS1; no longer U$21.CBUS0
- net GND: now also D7.A
- net MEGATXD: now also U$21.RXD; no longer U$21.TXD
Other:
- moved on the sheet: LED12, R28
Changed lines of the file:
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@@
 <layer number="56" name="wert" color="7" fill="1" visible="no" active="no"/>
 <layer number="57" name="tCAD" color="7" fill="1" visible="no" active="no"/>
+<layer number="58" name="bCAD" color="11" fill="1" visible="no" active="no"/>
 <layer number="59" name="tCarbon" color="7" fill="1" visible="no" active="no"/>
 <layer number="60" name="bCarbon" color="7" fill="1" visible="no" active="no"/>
@@
 <part name="GND80" library="supply1" deviceset="GND" device=""/>
 <part name="GND81" library="supply1" deviceset="GND" device=""/>
-<part name="LED12" library="adafruit" deviceset="LED" device="CHIP-LED0805" value="CBUS0"/>
+<part name="LED12" library="adafruit" deviceset="LED" device="CHIP-LED0805" value="CBUS1"/>
 <part name="R28" library="rcl" deviceset="R-US_" device="R0805" value="1k"/>
+<part name="P+16" library="supply1" deviceset="+5V" device=""/>
+<part name="GND39" library="supply1" deviceset="GND" device=""/>
+<part name="D7" library="diode" deviceset="ZENER-DIODE" device="DO41Z10"/>
 </parts>
 <sheets>
@@
 <instance part="GND80" gate="1" x="662.94" y="175.26"/>
 <instance part="GND81" gate="1" x="586.74" y="157.48"/>
-<instance part="LED12" gate="G$1" x="650.24" y="170.18" rot="R270"/>
-<instance part="R28" gate="G$1" x="673.1" y="170.18"/>
+<instance part="LED12" gate="G$1" x="650.24" y="167.64" rot="R270"/>
+<instance part="R28" gate="G$1" x="673.1" y="167.64"/>
+<instance part="P+16" gate="1" x="154.94" y="276.86"/>
+<instance part="GND39" gate="1" x="129.54" y="271.78"/>
+<instance part="D7" gate="G$1" x="142.24" y="274.32"/>
 </instances>
 <busses>
@@
 <junction x="596.9" y="162.56"/>
 </segment>
+<segment>
+<pinref part="GND39" gate="1" pin="GND"/>
+<wire x1="139.7" y1="274.32" x2="129.54" y2="274.32" width="0.1524" layer="91"/>
+<pinref part="D7" gate="G$1" pin="A"/>
+</segment>
 </net>
 <net name="+5V" class="0">
@@
 <pinref part="P+9" gate="1" pin="+5V"/>
 </segment>
+<segment>
+<pinref part="P+16" gate="1" pin="+5V"/>
+<wire x1="154.94" y1="274.32" x2="144.78" y2="274.32" width="0.1524" layer="91"/>
+<pinref part="D7" gate="G$1" pin="C"/>
+</segment>
 </net>
 <net name="ARD_D7" class="0">
@@
 <wire x1="248.92" y1="307.34" x2="243.84" y2="307.34" width="0.1524" layer="91"/>
 <pinref part="R5" gate="G$1" pin="2"/>
+<label x="248.92" y="307.34" size="1.778" layer="95"/>
 </segment>
 </net>
@@
 <wire x1="495.3" y1="139.7" x2="505.46" y2="139.7" width="0.1524" layer="91"/>
 <pinref part="U5" gate="A" pin="DP4"/>
+<label x="497.84" y="139.7" size="1.778" layer="95"/>
 </segment>
 </net>
@@
 <wire x1="495.3" y1="142.24" x2="505.46" y2="142.24" width="0.1524" layer="91"/>
 <pinref part="U5" gate="A" pin="DM4"/>
+<label x="497.84" y="142.24" size="1.778" layer="95"/>
 </segment>
 </net>
@@
 </segment>
 <segment>
-<wire x1="640.08" y1="182.88" x2="637.54" y2="182.88" width="0.1524" layer="91"/>
-<pinref part="U$21" gate="G$1" pin="TXD"/>
-<label x="637.794" y="183.388" size="1.778" layer="95"/>
+<wire x1="640.08" y1="180.34" x2="637.54" y2="180.34" width="0.1524" layer="91"/>
+<pinref part="U$21" gate="G$1" pin="RXD"/>
 </segment>
 </net>
@@
 <wire x1="505.46" y1="193.04" x2="495.3" y2="193.04" width="0.1524" layer="91"/>
 <pinref part="U5" gate="A" pin="DP1"/>
+<label x="497.84" y="193.04" size="1.778" layer="95"/>
 </segment>
 </net>
@@
 <wire x1="500.38" y1="195.58" x2="495.3" y2="195.58" width="0.1524" layer="91"/>
 <pinref part="U5" gate="A" pin="DM1"/>
+<label x="497.84" y="195.58" size="1.778" layer="95"/>
 </segment>
 </net>
@@
 </segment>
 </net>
-<net name="N$26" class="0">
+<net name="USB_RAW_5V" class="0">
 <segment>
 <pinref part="F3" gate="G$1" pin="2"/>
@@
 <wire x1="495.3" y1="160.02" x2="497.84" y2="160.02" width="0.1524" layer="91"/>
 <pinref part="U5" gate="A" pin="DM3"/>
+<label x="497.84" y="160.02" size="1.778" layer="95"/>
 </segment>
 </net>
@@
 </segment>
 <segment>
-<wire x1="683.26" y1="170.18" x2="678.18" y2="170.18" width="0.1524" layer="91"/>
+<wire x1="683.26" y1="167.64" x2="678.18" y2="167.64" width="0.1524" layer="91"/>
 <pinref part="R28" gate="G$1" pin="2"/>
 <label x="678.18" y="170.18" size="1.778" layer="95"/>
@@
 <net name="FT_CB0" class="0">
 <segment>
-<pinref part="U$21" gate="G$1" pin="CBUS0"/>
+<wire x1="645.16" y1="167.64" x2="637.54" y2="167.64" width="0.1524" layer="91"/>
+<pinref part="U$21" gate="G$1" pin="CBUS1"/>
 <pinref part="LED12" gate="G$1" pin="C"/>
-<wire x1="645.16" y1="170.18" x2="637.54" y2="170.18" width="0.1524" layer="91"/>
 </segment>
 </net>
@@
 <pinref part="LED12" gate="G$1" pin="A"/>
 <pinref part="R28" gate="G$1" pin="1"/>
-<wire x1="668.02" y1="170.18" x2="652.78" y2="170.18" width="0.1524" layer="91"/>
+<wire x1="668.02" y1="167.64" x2="652.78" y2="167.64" width="0.1524" layer="91"/>
 </segment>
 </net>

Commit message: labels
Parts:
- added C52: 100nF, rcl:C-USC0805
- added U$23: ESDTUDOR, adafruit:ESDTUDOR
Connections:
- net CP_DMINUS_TI renamed USB_CP_DMINUS_A
- net CP_DPLUS_TI renamed USB_CP_DPLUS_A
- net DMINUS_ASP renamed USB_ASP_DMINUS_A
- net DMINUS_HUB renamed USB_HUB_DMINUS_A
- net DMINUS_NEO_END renamed USB_NEO_DMINUS_B
- net DPLUS_ASP renamed USB_ASP_DPLUS_A
- net DPLUS_HUB renamed USB_HUB_DPLUS_A
- net DPLUS_NEO_END renamed USB_NEO_DPLUS_B
- net FT-DMINUS renamed USB_FT_DMINUS_B
- net FT-DPLUS renamed USB_FT_DPLUS_B
- net FT_DM renamed USB_FT_DMINUS_A
- net FT_DP renamed USB_FT_DPLUS_A
- net N$37 renamed USB_ASP_DPLUS_B
- net N$38 renamed USB_ASP_DMINUS_B
- net TUSB_DMINUS_POSTRES renamed USB_HUB_DMINUS_B
- net TUSB_DPLUS_POSTRES renamed USB_HUB_DPLUS_B
- net UBLOX_DMINUS renamed USB_NEO_DMINUS_A
- net UBLOX_DPLUS renamed USB_NEO_DPLUS_A
- net GND: now also C52.2
- net USB-3V3: now also C52.1
Other:
- note added: "run length-freq-ri"
Changed lines of the file:
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@@
 <part name="GND39" library="supply1" deviceset="GND" device=""/>
 <part name="D7" library="diode" deviceset="ZENER-DIODE" device="DO41Z10"/>
+<part name="C52" library="rcl" deviceset="C-US" device="C0805" value="100nF"/>
+<part name="GND90" library="supply1" deviceset="GND" device=""/>
+<part name="U$23" library="adafruit" deviceset="ESDTUDOR" device=""/>
 </parts>
 <sheets>
@@
 the BP pin and GND pin significantly reduces
 noise on the regulator output..."</text>
+<text x="424.18" y="205.74" size="1.778" layer="91">run length-freq-ri</text>
 </plain>
 <instances>
@@
 <instance part="GND39" gate="1" x="129.54" y="271.78"/>
 <instance part="D7" gate="G$1" x="142.24" y="274.32"/>
+<instance part="C52" gate="G$1" x="281.94" y="269.24"/>
+<instance part="GND90" gate="1" x="281.94" y="261.62"/>
+<instance part="U$23" gate="G$1" x="388.62" y="132.08"/>
 </instances>
 <busses>
@@
 <wire x1="139.7" y1="274.32" x2="129.54" y2="274.32" width="0.1524" layer="91"/>
 <pinref part="D7" gate="G$1" pin="A"/>
+</segment>
+<segment>
+<pinref part="C52" gate="G$1" pin="2"/>
+<pinref part="GND90" gate="1" pin="GND"/>
 </segment>
 </net>
@@
 </segment>
 </net>
-<net name="UBLOX_DPLUS" class="0">
+<net name="USB_NEO_DPLUS_A" class="0">
 <segment>
 <wire x1="266.7" y1="266.7" x2="261.62" y2="266.7" width="0.1524" layer="91"/>
@@
 </segment>
 </net>
-<net name="UBLOX_DMINUS" class="0">
+<net name="USB_NEO_DMINUS_A" class="0">
 <segment>
 <wire x1="266.7" y1="261.62" x2="261.62" y2="261.62" width="0.1524" layer="91"/>
@@
 </segment>
 </net>
-<net name="DPLUS_NEO_END" class="0">
+<net name="USB_NEO_DPLUS_B" class="0">
 <segment>
 <pinref part="R2" gate="G$1" pin="1"/>
@@
 </segment>
 </net>
-<net name="DMINUS_NEO_END" class="0">
+<net name="USB_NEO_DMINUS_B" class="0">
 <segment>
 <pinref part="R5" gate="G$1" pin="1"/>
@@
 </segment>
 </net>
-<net name="N$37" class="0">
+<net name="USB_ASP_DPLUS_B" class="0">
 <segment>
 <pinref part="R19" gate="G$1" pin="1"/>
@@
 </segment>
 </net>
-<net name="N$38" class="0">
+<net name="USB_ASP_DMINUS_B" class="0">
 <segment>
 <pinref part="R18" gate="G$1" pin="1"/>
@@
 </segment>
 </net>
-<net name="FT-DPLUS" class="0">
+<net name="USB_FT_DPLUS_B" class="0">
 <segment>
 <pinref part="C34" gate="G$1" pin="1"/>
@@
 </segment>
 </net>
-<net name="FT-DMINUS" class="0">
+<net name="USB_FT_DMINUS_B" class="0">
 <segment>
 <wire x1="609.6" y1="142.24" x2="617.22" y2="142.24" width="0.1524" layer="91"/>
@@
 </segment>
 </net>
-<net name="FT_DM" class="0">
+<net name="USB_FT_DMINUS_A" class="0">
 <segment>
 <wire x1="645.16" y1="142.24" x2="650.24" y2="142.24" width="0.1524" layer="91"/>
@@
 </segment>
 </net>
-<net name="FT_DP" class="0">
+<net name="USB_FT_DPLUS_A" class="0">
 <segment>
 <wire x1="642.62" y1="139.7" x2="650.24" y2="139.7" width="0.1524" layer="91"/>
@@
 </segment>
 </net>
-<net name="DPLUS_ASP" class="0">
+<net name="USB_ASP_DPLUS_A" class="0">
 <segment>
 <wire x1="101.6" y1="27.94" x2="119.38" y2="27.94" width="0.1524" layer="91"/>
@@
 </segment>
 </net>
-<net name="DMINUS_ASP" class="0">
+<net name="USB_ASP_DMINUS_A" class="0">
 <segment>
 <pinref part="R18" gate="G$1" pin="2"/>
@@
 </segment>
 </net>
-<net name="DPLUS_HUB" class="0">
+<net name="USB_HUB_DPLUS_A" class="0">
 <segment>
 <wire x1="421.64" y1="165.1" x2="444.5" y2="165.1" width="0.1524" layer="91"/>
@@
 </segment>
 </net>
-<net name="DMINUS_HUB" class="0">
+<net name="USB_HUB_DMINUS_A" class="0">
 <segment>
 <wire x1="431.8" y1="167.64" x2="444.5" y2="167.64" width="0.1524" layer="91"/>
@@
 </segment>
 <segment>
-<wire x1="264.16" y1="271.78" x2="261.62" y2="271.78" width="0.1524" layer="91"/>
+<wire x1="307.34" y1="271.78" x2="281.94" y2="271.78" width="0.1524" layer="91"/>
 <pinref part="U$2" gate="G$1" pin="7_VDDUSB"/>
 <label x="261.62" y="271.78" size="1.778" layer="95"/>
+<pinref part="C52" gate="G$1" pin="1"/>
+<wire x1="281.94" y1="271.78" x2="261.62" y2="271.78" width="0.1524" layer="91"/>
+<junction x="281.94" y="271.78"/>
 </segment>
 <segment>
@@
 </segment>
 </net>
-<net name="TUSB_DMINUS_POSTRES" class="0">
+<net name="USB_HUB_DMINUS_B" class="0">
 <segment>
 <wire x1="114.3" y1="81.28" x2="134.62" y2="81.28" width="0.1524" layer="91"/>
@@
 </segment>
 </net>
-<net name="TUSB_DPLUS_POSTRES" class="0">
+<net name="USB_HUB_DPLUS_B" class="0">
 <segment>
 <wire x1="124.46" y1="83.82" x2="134.62" y2="83.82" width="0.1524" layer="91"/>
@@
 </segment>
 </net>
-<net name="CP_DMINUS_TI" class="0">
+<net name="USB_CP_DMINUS_A" class="0">
 <segment>
 <wire x1="408.94" y1="279.4" x2="429.26" y2="279.4" width="0.1524" layer="91"/>
@@
 </segment>
 </net>
-<net name="CP_DPLUS_TI" class="0">
+<net name="USB_CP_DPLUS_A" class="0">
 <segment>
 <wire x1="408.94" y1="284.48" x2="429.26" y2="284.48" width="0.1524" layer="91"/>
